Commit message: gripper bug

File: Robots/onrobot_rg_description/urdf/onrobot_rg2.urdf (robot description, URDF)
Before this commit: robot rg2, 7 links, 6 joints
Joints:
- joint right_inner_knuckle_joint: origin xyz=0 -0.007678 0.1422970 rpy=0 0 -3.14159 -> xyz=0 0.007678 0.1422970 rpy=0 0 -3.14159
